Commit message: ---------prsg2_params.yaml------- Set wheel_track to 0.203. Change IR plan for my robot. Comment out ir_left_link and ir_right_link, change R pins. Add ir_rear_link sensor. ---------prsg2_description.xacro------- Set ir_setback to 0. Comment out ir_left_link and ir_right_link. Add ir_rear_link. Comment out camera.

File: urdf/prsg2_description.xacro (robot description, xacro)
@@ -13,5 +13,5 @@
   <xacro:property name="caster_thickness" value="0.012" />
   <xacro:property name="caster_setback" value="${caster_diameter / 2}" />
-  <xacro:property name="ir_setback" value="0.015" />
+  <xacro:property name="ir_setback" value="0.00" />
   <xacro:property name="camera_height" value="0.075" />
   <xacro:property name="camera_setback" value="0.025" />
@@ -91,9 +91,15 @@
       l0="base_link" l1="${link_name}" />
   </xacro:macro>
+  <!--
   <xacro:ir_sensor link_name="ir_left_link" theta="${90 * degree}" />
+  -->
   <xacro:ir_sensor link_name="ir_left_front_link" theta="${45 * degree}" />
   <xacro:ir_sensor link_name="ir_front_link" theta="${0 * degree}" />
   <xacro:ir_sensor link_name="ir_right_front_link" theta="${-45 * degree}" />
+  <!--
   <xacro:ir_sensor link_name="ir_right_link" theta="${-90 * degree}" />
+  -->
+  <xacro:ir_sensor link_name="ir_rear_link" theta="${180 * degree}" />
+  <!-- No camera
   <link name="camera_link">
     <visual>
@@ -109,3 +115,4 @@
   <xacro:polar_position r="${base_diameter/2 - camera_setback}" theta="0"
     z="${deck_height + camera_height}" l0="base_link" l1="camera_link" />
+  -->
 </robot>

Commit message: Add changes for my robot.

File: urdf/prsg2_description.xacro (robot description, xacro)
@@ -5,11 +5,11 @@
   <xacro:property name="inch" value="0.0254" />
   <xacro:property name="base_diameter" value="${9 * inch}" />
-  <xacro:property name="base_thickness" value="0.008" />
-  <xacro:property name="deck_height" value="0.050" />
-  <xacro:property name="wheel_diameter" value="0.060" />
-  <xacro:property name="wheel_thickness" value="0.008" />
-  <xacro:property name="wheel_separation" value="0.203" />
-  <xacro:property name="caster_diameter" value="0.029" />
-  <xacro:property name="caster_thickness" value="0.012" />
+  <xacro:property name="base_thickness" value="0.005" />
+  <xacro:property name="deck_height" value="0.0206" />
+  <xacro:property name="wheel_diameter" value="0.070" />
+  <xacro:property name="wheel_thickness" value="0.00635" />
+  <xacro:property name="wheel_separation" value="0.206375" />
+  <xacro:property name="caster_diameter" value="0.014" />
+  <xacro:property name="caster_thickness" value="0.014" />
   <xacro:property name="caster_setback" value="${caster_diameter / 2}" />
   <xacro:property name="ir_setback" value="0.00" />
@@ -91,13 +91,9 @@
       l0="base_link" l1="${link_name}" />
   </xacro:macro>
-  <!--
-  <xacro:ir_sensor link_name="ir_left_link" theta="${90 * degree}" />
-  -->
-  <xacro:ir_sensor link_name="ir_left_front_link" theta="${45 * degree}" />
+  <xacro:ir_sensor link_name="ir_left_link" theta="${70 * degree}" angle="${20 *degree}" />
+  <xacro:ir_sensor link_name="ir_left_front_link" theta="${52 * degree}" />
   <xacro:ir_sensor link_name="ir_front_link" theta="${0 * degree}" />
-  <xacro:ir_sensor link_name="ir_right_front_link" theta="${-45 * degree}" />
-  <!--
-  <xacro:ir_sensor link_name="ir_right_link" theta="${-90 * degree}" />
-  -->
+  <xacro:ir_sensor link_name="ir_right_front_link" theta="${-52 * degree}" />
+  <xacro:ir_sensor link_name="ir_right_link" theta="${-70 * degree}" angle="${-20 * degree}" />
   <xacro:ir_sensor link_name="ir_rear_link" theta="${180 * degree}" />
   <!-- No camera
